File: POS_router/GT_pos_router.brd (EAGLE design)
At the start: 86.8 x 70 mm, 75 parts, among them J1 DB25-RA-MALE, J10 HDR_1X4, J2 DB25-RA-FEMALE, J3 RPI_ZERO_HDR0.2_STACK, J4 PWR_JACK_SW_NC, J7 RJ45-JACK-VERT, J8 USB-MICRO-B-SMT-FLG, J9 USB-A-RECEPT-RA, U1 FT2232H, U2 MAX3243ST-EB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

Commit message: Moved RJ45 to edge and made RA
Parts:
- removed J7: RJ45-JACK-VERT, mechanical:RJ45-VERT
- added J5: RJ45-JACKRA, mechanical:RJ45-RA
- moved R15 60.9 mm to (18.2, 66.2)
- moved R14 53.2 mm to (22.3, 57.3)
- moved R12 50.8 mm to (43.1, 65.3)
- moved R13 46.2 mm to (39.7, 60.9), turned to 180 degrees
- moved J2 5.71 mm to (76.0, 18.4)
Connections:
- net 24V: now also J5.1; no longer J7.1
- net BUFF_CSN: now also J5.8; no longer J7.8
- net BUFF_MISO: now also J5.4; no longer J7.4
- net BUFF_MOSI: now also J5.7; no longer J7.7
- net BUFF_SCLK: now also J5.3; no longer J7.3
- net GND: now also J5.2; no longer J7.2
- net SCR_BUTTN: now also J5.5; no longer J7.5
- net SCR_LEDN: now also J5.6; no longer J7.6
Routing:
- net 24V: track 50.0 -> 122.4 mm
- net SCR_LEDN: track 71.3 -> 13.5 mm, vias 1 -> 0
- net SCR_CSN: track 76.1 -> 31.6 mm, vias 1 -> 0
- net PI_MISO: track 126.4 -> 83.1 mm
- net PI_MOSI: track 130.1 -> 88.6 mm
- net PI_SCLK: track 114.5 -> 81.8 mm, vias 3 -> 2
- net SCR_BUTTN: track 61.3 -> 29.4 mm
- net 5V: track 168.9 -> 188.3 mm
- net POS_TD: track 36.1 -> 27.9 mm
- net BUFF_MISO: track 2.38 -> 10.4 mm
- net BUFF_CSN: track 3.21 -> 11.0 mm, vias 0 -> 1
- net BUFF_SCLK: track 6.37 -> 12.8 mm
- net POS_RD: track 34.8 -> 28.9 mm, vias 2 -> 1
- net POS_DTR: track 34.9 -> 29.2 mm
- net POS_CTS: track 30.9 -> 25.2 mm
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